Commit message: Update RGB-D camera simulation

File: src/jaka_description/urdf/jaka_zu3_tools.xacro (robot description, xacro)
@@ -28,4 +28,23 @@
       <child link="camera_link"/>
       <origin xyz="0 0 0.015" rpy="-1.57079632679 -1.57079632679 0"/>
+    </joint>
+    <link name="camera_test_cube_link">
+      <inertial>
+        <mass value="0.001"/>
+        <inertia ixx="0.000000417" ixy="0" ixz="0" iyy="0.000000417" iyz="0" izz="0.000000417"/>
+      </inertial>
+      <visual>
+        <geometry>
+          <box size="0.05 0.05 0.05"/>
+        </geometry>
+        <material name="test_cube_red">
+          <color rgba="1 0 0 1"/>
+        </material>
+      </visual>
+    </link>
+    <joint name="camera_test_cube_joint" type="fixed">
+      <parent link="${parent}"/>
+      <child link="camera_test_cube_link"/>
+      <origin xyz="0 0 0.30" rpy="0 0 0"/>
     </joint>
     <link name="camera_optical_frame"/>

Commit message: Add RGB-D target detection and world coordinate estimation

File: src/jaka_description/urdf/jaka_zu3_tools.xacro (robot description, xacro)
@@ -29,28 +29,9 @@
       <origin xyz="0 0 0.015" rpy="-1.57079632679 -1.57079632679 0"/>
     </joint>
-    <link name="camera_test_cube_link">
-      <inertial>
-        <mass value="0.001"/>
-        <inertia ixx="0.000000417" ixy="0" ixz="0" iyy="0.000000417" iyz="0" izz="0.000000417"/>
-      </inertial>
-      <visual>
-        <geometry>
-          <box size="0.05 0.05 0.05"/>
-        </geometry>
-        <material name="test_cube_red">
-          <color rgba="1 0 0 1"/>
-        </material>
-      </visual>
-    </link>
-    <joint name="camera_test_cube_joint" type="fixed">
-      <parent link="${parent}"/>
-      <child link="camera_test_cube_link"/>
-      <origin xyz="0 0 0.30" rpy="0 0 0"/>
-    </joint>
     <link name="camera_optical_frame"/>
     <joint name="camera_optical_joint" type="fixed">
       <parent link="camera_link"/>
       <child link="camera_optical_frame"/>
-      <origin xyz="0.04 0 0" rpy="-1.57079632679 0 -1.57079632679"/>
+      <origin xyz="0 0 0" rpy="-1.57079632679 0 -1.57079632679"/>
     </joint>
     <xacro:if value="${use_gazebo and enable_camera_sensor}">
@@ -58,5 +39,5 @@
         <!-- Keep both aligned image streams inexpensive enough for ros2_control. -->
         <sensor name="wrist_depth_camera" type="depth_camera">
-          <pose>0.014 0 0 0 0 0</pose>
+          <pose>0.02 0 0 0 0 0</pose>
           <always_on>true</always_on>
           <update_rate>5</update_rate>

Commit message: 更新加入了二指夹爪，视觉抓取功能

File: src/jaka_description/urdf/jaka_zu3_tools.xacro (robot description, xacro)
@@ -27,5 +27,5 @@
       <parent link="${parent}"/>
       <child link="camera_link"/>
-      <origin xyz="0 0 0.015" rpy="-1.57079632679 -1.57079632679 0"/>
+      <origin xyz="0 -0.05 -0.02" rpy="-1.57079632679 -1.57079632679 0"/>
     </joint>
     <link name="camera_optical_frame"/>
@@ -79,3 +79,87 @@
     </xacro:if>
   </xacro:macro>
+  <xacro:macro name="jaka_zu3_parallel_gripper" params="parent">
+    <material name="gripper_black">
+      <color rgba="0.08 0.08 0.08 1"/>
+    </material>
+    <material name="finger_red">
+      <color rgba="0.65 0.12 0.08 1"/>
+    </material>
+    <link name="gripper_base_link">
+      <inertial>
+        <mass value="0.12"/>
+        <inertia ixx="0.0001" ixy="0" ixz="0" iyy="0.0001" iyz="0" izz="0.0001"/>
+      </inertial>
+      <visual>
+        <geometry>
+          <box size="0.06 0.06 0.035"/>
+        </geometry>
+        <material name="gripper_black"/>
+      </visual>
+      <collision>
+        <geometry>
+          <box size="0.06 0.06 0.03"/>
+        </geometry>
+      </collision>
+    </link>
+    <joint name="gripper_base_joint" type="fixed">
+      <parent link="${parent}"/>
+      <child link="gripper_base_link"/>
+      <origin xyz="0 0 0.02" rpy="0 0 1.5708"/>
+    </joint>
+    <link name="left_finger_link">
+      <inertial>
+        <mass value="0.03"/>
+        <inertia ixx="0.00002" ixy="0" ixz="0" iyy="0.00002" iyz="0" izz="0.00002"/>
+      </inertial>
+      <visual>
+        <geometry>
+          <box size="0.03 0.01 0.04"/>
+        </geometry>
+        <material name="finger_red"/>
+      </visual>
+      <collision>
+        <geometry>
+          <box size="0.03 0.01 0.04"/>
+        </geometry>
+      </collision>
+    </link>
+    <joint name="left_finger_joint" type="prismatic">
+      <parent link="gripper_base_link"/>
+      <child link="left_finger_link"/>
+      <origin xyz="0 0.025 0.04" rpy="0 0 0"/>
+      <axis xyz="0 -1 0"/>
+      <limit lower="0" upper="0.025" effort="20" velocity="0.2"/>
+    </joint>
+    <link name="right_finger_link">
+      <inertial>
+        <mass value="0.03"/>
+        <inertia ixx="0.00002" ixy="0" ixz="0" iyy="0.00002" iyz="0" izz="0.00002"/>
+      </inertial>
+      <visual>
+        <geometry>
+          <box size="0.03 0.01 0.04"/>
+        </geometry>
+        <material name="finger_red"/>
+      </visual>
+      <collision>
+        <geometry>
+          <box size="0.03 0.01 0.04"/>
+        </geometry>
+      </collision>
+    </link>
+    <joint name="right_finger_joint" type="prismatic">
+      <parent link="gripper_base_link"/>
+      <child link="right_finger_link"/>
+      <origin xyz="0 -0.025 0.04" rpy="0 0 0"/>
+      <axis xyz="0 1 0"/>
+      <limit lower="0" upper="0.025" effort="20" velocity="0.2"/>
+    </joint>
+    <link name="gripper_tcp"/>
+    <joint name="gripper_tcp_joint" type="fixed">
+      <parent link="gripper_base_link"/>
+      <child link="gripper_tcp"/>
+      <origin xyz="0 0 -0.105" rpy="0 0 0"/>
+    </joint>
+  </xacro:macro>
 </robot>

File: src/jaka_zu3_moveit_config/config/jaka_zu3.ros2_control.xacro (robot description, xacro)
@@ -56,4 +56,6 @@
                 <state_interface name="velocity"/>
             </joint>
+            <joint name="left_finger_joint"><command_interface name="position"/><state_interface name="position"><param name="initial_value">0.0</param></state_interface><state_interface name="velocity"/></joint>
+            <joint name="right_finger_joint"><command_interface name="position"/><state_interface name="position"><param name="initial_value">0.0</param></state_interface><state_interface name="velocity"/></joint>
         </ros2_control>
     </xacro:macro>

File: src/jaka_zu3_moveit_config/config/jaka_zu3.urdf.xacro (robot description, xacro)
@@ -15,4 +15,5 @@
         use_gazebo="$(arg use_gazebo)"
         enable_camera_sensor="$(arg enable_camera_sensor)" />
+    <xacro:jaka_zu3_parallel_gripper parent="Link_6" />
     <!-- 加载 ros2_control 配置 -->
     <xacro:jaka_zu3_ros2_control name="jaka_zu3_hardware" initial_positions_file="$(arg initial_positions_file)" use_gazebo="$(arg use_gazebo)" use_rviz_sim="$(arg use_rviz_sim)" />

Commit message: Update vision grasp simulation

File: src/jaka_description/urdf/jaka_zu3_tools.xacro (robot description, xacro)
@@ -79,5 +79,5 @@
     </xacro:if>
   </xacro:macro>
-  <xacro:macro name="jaka_zu3_parallel_gripper" params="parent">
+  <xacro:macro name="jaka_zu3_parallel_gripper" params="parent use_gazebo:=false">
     <material name="gripper_black">
       <color rgba="0.08 0.08 0.08 1"/>
@@ -115,18 +115,25 @@
       <visual>
         <geometry>
-          <box size="0.03 0.01 0.04"/>
+          <box size="0.06 0.01 0.04"/>
         </geometry>
         <material name="finger_red"/>
       </visual>
-      <collision>
-        <geometry>
-          <box size="0.03 0.01 0.04"/>
-        </geometry>
-      </collision>
+      <!-- In Gazebo the object is attached only after a verified close.  A
+           finger collision here can pin the first finger that touches an
+           off-centre cube, making a symmetric gripper appear one-sided. -->
+      <xacro:unless value="${use_gazebo}">
+        <collision>
+          <geometry>
+            <box size="0.06 0.01 0.04"/>
+          </geometry>
+        </collision>
+      </xacro:unless>
     </link>
     <joint name="left_finger_joint" type="prismatic">
       <parent link="gripper_base_link"/>
       <child link="left_finger_link"/>
-      <origin xyz="0 0.025 0.04" rpy="0 0 0"/>
+      <!-- At zero travel the inner faces are 70 mm apart, enough to clear
+           the 50 mm target. Positive travel closes both fingers inward. -->
+      <origin xyz="0 0.040 0.04" rpy="0 0 0"/>
       <axis xyz="0 -1 0"/>
       <limit lower="0" upper="0.025" effort="20" velocity="0.2"/>
@@ -139,18 +146,20 @@
       <visual>
         <geometry>
-          <box size="0.03 0.01 0.04"/>
+          <box size="0.06 0.01 0.04"/>
         </geometry>
         <material name="finger_red"/>
       </visual>
-      <collision>
-        <geometry>
-          <box size="0.03 0.01 0.04"/>
-        </geometry>
-      </collision>
+      <xacro:unless value="${use_gazebo}">
+        <collision>
+          <geometry>
+            <box size="0.06 0.01 0.04"/>
+          </geometry>
+        </collision>
+      </xacro:unless>
     </link>
     <joint name="right_finger_joint" type="prismatic">
       <parent link="gripper_base_link"/>
       <child link="right_finger_link"/>
-      <origin xyz="0 -0.025 0.04" rpy="0 0 0"/>
+      <origin xyz="0 -0.040 0.04" rpy="0 0 0"/>
       <axis xyz="0 1 0"/>
       <limit lower="0" upper="0.025" effort="20" velocity="0.2"/>
@@ -162,4 +171,12 @@
       <origin xyz="0 0 -0.105" rpy="0 0 0"/>
     </joint>
+    <gazebo reference="left_finger_link">
+      <mu1>2.0</mu1>
+      <mu2>2.0</mu2>
+    </gazebo>
+    <gazebo reference="right_finger_link">
+      <mu1>2.0</mu1>
+      <mu2>2.0</mu2>
+    </gazebo>
   </xacro:macro>
 </robot>

File: src/jaka_zu3_moveit_config/config/jaka_zu3.urdf.xacro (robot description, xacro)
@@ -5,4 +5,5 @@
     <xacro:arg name="use_rviz_sim" default="false"/>
     <xacro:arg name="enable_camera_sensor" default="true"/>
+    <xacro:arg name="enable_grasp_attachment" default="false"/>
     <!-- Import jaka_zu3 urdf file -->
     <xacro:include filename="$(find jaka_description)/urdf/jaka_zu3.urdf" />
@@ -15,5 +16,7 @@
         use_gazebo="$(arg use_gazebo)"
         enable_camera_sensor="$(arg enable_camera_sensor)" />
-    <xacro:jaka_zu3_parallel_gripper parent="Link_6" />
+    <xacro:jaka_zu3_parallel_gripper
+        parent="Link_6"
+        use_gazebo="$(arg use_gazebo)" />
     <!-- 加载 ros2_control 配置 -->
     <xacro:jaka_zu3_ros2_control name="jaka_zu3_hardware" initial_positions_file="$(arg initial_positions_file)" use_gazebo="$(arg use_gazebo)" use_rviz_sim="$(arg use_rviz_sim)" />
@@ -22,8 +25,25 @@
         <gazebo>
             <plugin filename="gz_ros2_control-system"
-        name="gz_ros2_control::GazeboSimROS2ControlPlugin">
+                    name="gz_ros2_control::GazeboSimROS2ControlPlugin">
                 <parameters>$(find jaka_zu3_moveit_config)/config/ros2_controllers.yaml</parameters>
             </plugin>
         </gazebo>
+        <!-- Gazebo contact friction alone is not reliable enough to keep a
+             small object between two position-controlled fingers.  Enable a
+             fixed attachment only for the guarded demo pick; target_motion
+             detaches it at startup and attaches it after both fingers close. -->
+        <xacro:if value="$(arg enable_grasp_attachment)">
+            <gazebo>
+                <plugin filename="ignition-gazebo-detachable-joint-system"
+                        name="ignition::gazebo::systems::DetachableJoint">
+                    <parent_link>Link_6</parent_link>
+                    <child_model>target_cube</child_model>
+                    <child_link>link</child_link>
+                    <detach_topic>/gripper/detach</detach_topic>
+                    <attach_topic>/gripper/attach</attach_topic>
+                    <output_topic>/gripper/attached</output_topic>
+                </plugin>
+            </gazebo>
+        </xacro:if>
     </xacro:if>
 </robot>

Commit message: update vision grasping project

File: src/jaka_description/urdf/jaka_zu3_tools.xacro (robot description, xacro)
@@ -119,23 +119,26 @@
         <material name="finger_red"/>
       </visual>
-      <!-- In Gazebo the object is attached only after a verified close.  A
-           finger collision here can pin the first finger that touches an
-           off-centre cube, making a symmetric gripper appear one-sided. -->
-      <xacro:unless value="${use_gazebo}">
-        <collision>
-          <geometry>
-            <box size="0.06 0.01 0.04"/>
-          </geometry>
-        </collision>
-      </xacro:unless>
+      <!-- Keep contact geometry while commanding both finger joints from
+           the same trajectory; verify their measured positions before lift. -->
+      <collision>
+        <geometry>
+          <box size="0.06 0.01 0.04"/>
+        </geometry>
+      </collision>
     </link>
     <joint name="left_finger_joint" type="prismatic">
       <parent link="gripper_base_link"/>
       <child link="left_finger_link"/>
+      <!-- Both simulated joints receive the same position trajectory. The
+           legacy Gazebo mimic follower can lag when a finger makes contact. -->
       <!-- At zero travel the inner faces are 70 mm apart, enough to clear
            the 50 mm target. Positive travel closes both fingers inward. -->
       <origin xyz="0 0.040 0.04" rpy="0 0 0"/>
       <axis xyz="0 -1 0"/>
-      <limit lower="0" upper="0.025" effort="20" velocity="0.2"/>
+      <!-- Keep the commanded open position (0) inside the physics limits.
+           Starting exactly on the hard stop pins the first close in this
+           Gazebo setup. Use the same interior open pose for every transfer.
+           This 1 mm margin is not part of the commanded finger stroke. -->
+      <limit lower="-0.001" upper="0.025" effort="20" velocity="0.2"/>
     </joint>
     <link name="right_finger_link">
@@ -150,11 +153,9 @@
         <material name="finger_red"/>
       </visual>
-      <xacro:unless value="${use_gazebo}">
-        <collision>
-          <geometry>
-            <box size="0.06 0.01 0.04"/>
-          </geometry>
-        </collision>
-      </xacro:unless>
+      <collision>
+        <geometry>
+          <box size="0.06 0.01 0.04"/>
+        </geometry>
+      </collision>
     </link>
     <joint name="right_finger_joint" type="prismatic">
@@ -163,5 +164,6 @@
       <origin xyz="0 -0.040 0.04" rpy="0 0 0"/>
       <axis xyz="0 1 0"/>
-      <limit lower="0" upper="0.025" effort="20" velocity="0.2"/>
+      <!-- Same hard-stop margin as the left joint; open commands remain 0. -->
+      <limit lower="-0.001" upper="0.025" effort="20" velocity="0.2"/>
     </joint>
     <link name="gripper_tcp"/>

File: src/jaka_zu3_moveit_config/config/jaka_zu3.ros2_control.xacro (robot description, xacro)
@@ -56,5 +56,13 @@
                 <state_interface name="velocity"/>
             </joint>
-            <joint name="left_finger_joint"><command_interface name="position"/><state_interface name="position"><param name="initial_value">0.0</param></state_interface><state_interface name="velocity"/></joint>
+            <!-- Drive both fingers with the same trajectory and expose both
+                 measured states, including while either finger is in contact. -->
+            <joint name="left_finger_joint">
+                <command_interface name="position"/>
+                <state_interface name="position">
+                    <param name="initial_value">0.0</param>
+                </state_interface>
+                <state_interface name="velocity"/>
+            </joint>
             <joint name="right_finger_joint"><command_interface name="position"/><state_interface name="position"><param name="initial_value">0.0</param></state_interface><state_interface name="velocity"/></joint>
         </ros2_control>

Commit message: update visual grasp demo and documentation

File: src/jaka_description/urdf/jaka_zu3_tools.xacro (robot description, xacro)
@@ -119,9 +119,10 @@
         <material name="finger_red"/>
       </visual>
-      <!-- Keep contact geometry while commanding both finger joints from
-           the same trajectory; verify their measured positions before lift. -->
+      <!-- The visual finger reaches the ground when gripper_base_link is at
+           z=0.06. Inset the collision by 2 mm at each end so Gazebo ground
+           friction cannot pin the prismatic joint during lateral closing. -->
       <collision>
         <geometry>
-          <box size="0.06 0.01 0.04"/>
+          <box size="0.06 0.01 0.036"/>
         </geometry>
       </collision>
@@ -132,7 +133,7 @@
       <!-- Both simulated joints receive the same position trajectory. The
            legacy Gazebo mimic follower can lag when a finger makes contact. -->
-      <!-- At zero travel the inner faces are 70 mm apart, enough to clear
-           the 50 mm target. Positive travel closes both fingers inward. -->
-      <origin xyz="0 0.040 0.04" rpy="0 0 0"/>
+      <!-- At zero travel the inner faces are 40 mm apart, enough to clear
+           the 20 mm target. Positive travel closes both fingers inward. -->
+      <origin xyz="0 0.025 0.04" rpy="0 0 0"/>
       <axis xyz="0 -1 0"/>
       <!-- Keep the commanded open position (0) inside the physics limits.
@@ -140,5 +141,5 @@
            Gazebo setup. Use the same interior open pose for every transfer.
            This 1 mm margin is not part of the commanded finger stroke. -->
-      <limit lower="-0.001" upper="0.025" effort="20" velocity="0.2"/>
+      <limit lower="-0.001" upper="0.011" effort="20" velocity="0.2"/>
     </joint>
     <link name="right_finger_link">
@@ -153,7 +154,8 @@
         <material name="finger_red"/>
       </visual>
+      <!-- Match the left finger's 2 mm ground-contact clearance. -->
       <collision>
         <geometry>
-          <box size="0.06 0.01 0.04"/>
+          <box size="0.06 0.01 0.036"/>
         </geometry>
       </collision>
@@ -162,8 +164,8 @@
       <parent link="gripper_base_link"/>
       <child link="right_finger_link"/>
-      <origin xyz="0 -0.040 0.04" rpy="0 0 0"/>
+      <origin xyz="0 -0.025 0.04" rpy="0 0 0"/>
       <axis xyz="0 1 0"/>
       <!-- Same hard-stop margin as the left joint; open commands remain 0. -->
-      <limit lower="-0.001" upper="0.025" effort="20" velocity="0.2"/>
+      <limit lower="-0.001" upper="0.011" effort="20" velocity="0.2"/>
     </joint>
     <link name="gripper_tcp"/>
